Commit message: fixing root links

File: catkin_ws/src/my_robot/urdf/my_robot.xacro (robot description, xacro)
@@ -6,6 +6,4 @@
     <parent link="robot_footprint"/>
     <child link="chassis" />
-    <child link="left_wheel" />
-    <child link="right_wheel" />
   </joint>
 <!-- robot chasis -->
@@ -58,4 +56,9 @@
     </visual>
   </link>
+<joint name="robot_right_wheel_joint" type="fixed">
+  <origin xyz="0 0 0" rpy="0 0 0"/>
+  <parent link="chasis"/>
+  <child link="right_wheel"/>
+</joint>
 <!-- right side wheel -->
   <link name="right_wheel">
@@ -80,4 +83,9 @@
     </collision>
   </link>
+<joint name="robot_left_wheel_joint" type="fixed">
+  <origin xyz="0 0 0" rpy="0 0 0"/>
+  <parent link="chasis"/>
+  <child link="left_wheel"/>
+</joint>
 <!-- left side wheel -->
   <link name="left_wheel">
@@ -110,5 +118,5 @@
     <dynamics damping="1.0" friction="1.0"/>
   </joint>
-<joint type="continuous" name="right_wheel_hinge">
+ <joint type="continuous" name="right_wheel_hinge">
     <origin xyz="0 0.15 0" rpy="0 0 0"/>
     <child link="left_wheel"/>

Commit message: adding camera lidar sensor

File: catkin_ws/src/my_robot/urdf/my_robot.xacro (robot description, xacro)
@@ -126,3 +126,8 @@
     <dynamics damping="1.0" friction="1.0"/>
   </joint>
+ <joint name="camera_joint" type="fixed">
+  <origin xyz="0 0 0" rpy="0 0 0"/>
+  <parent link="chasis"/>
+  <child link="left_wheel"/>
+</joint>
 </robot>

Commit message: adding sensors and updating launch file

File: catkin_ws/src/my_robot/urdf/my_robot.xacro (robot description, xacro)
@@ -1,4 +1,5 @@
 <?xml version='1.0'?>
 <robot name="my_robot" xmlns:xacro="http://www.ros.org/wiki/xacro">
+  <xacro:include filename="$(find my_robot)/urdf/my_robot.gazebo" />
   <link name="robot_footprint"></link>
   <joint name="robot_footprint_joint" type="fixed">
@@ -8,5 +9,5 @@
   </joint>
 <!-- robot chasis -->
-  <link name='chassis'>
+  <link name="chassis">
     <pose>0 0 0.1 0 0 0</pose>
     <inertial>
@@ -19,5 +20,5 @@
       />
     </inertial>
-    <collision name='collision'>
+    <collision name="collision">
       <origin xyz="0 0 0" rpy=" 0 0 0"/>
       <geometry>
@@ -25,5 +26,5 @@
       </geometry>
     </collision>
-    <visual name='chassis_visual'>
+    <visual name="chassis_visual">
       <origin xyz="0 0 0" rpy=" 0 0 0"/>
       <geometry>
@@ -31,5 +32,5 @@
       </geometry>
     </visual>
-    <collision name='back_caster_collision'>
+    <collision name="back_caster_collision">
       <origin xyz="-0.15 0 -0.05" rpy=" 0 0 0"/>
       <geometry>
@@ -37,5 +38,5 @@
       </geometry>
     </collision>
-    <visual name='back_caster_visual'>
+    <visual name="back_caster_visual">
       <origin xyz="-0.15 0 -0.05" rpy=" 0 0 0"/>
       <geometry>
@@ -43,5 +44,5 @@
       </geometry>
     </visual>
-    <collision name='front_caster_collision'>
+    <collision name="front_caster_collision">
       <origin xyz="0.15 0 -0.05" rpy=" 0 0 0"/>
       <geometry>
@@ -49,5 +50,5 @@
       </geometry>
     </collision>
-    <visual name='front_caster_visual'>
+    <visual name="front_caster_visual">
       <origin xyz="0.15 0 -0.05" rpy=" 0 0 0"/>
       <geometry>
@@ -56,15 +57,12 @@
     </visual>
   </link>
-<joint name="robot_right_wheel_joint" type="fixed">
-  <origin xyz="0 0 0" rpy="0 0 0"/>
-  <parent link="chasis"/>
-  <child link="right_wheel"/>
-</joint>
 <!-- right side wheel -->
   <link name="right_wheel">
     <inertial>
+      <mass value="5"/>
       <origin xyz="0 0 0" rpy="0 1.5707 1.5707"/>
       <mass value="5.0"/>
-      <inertia  ixx="0.1" ixy="0" ixz="0"
+      <inertia
+            ixx="0.1" ixy="0" ixz="0"
             iyy="0.1" iyz="0"
             izz="0.1"/>
@@ -83,12 +81,8 @@
     </collision>
   </link>
-<joint name="robot_left_wheel_joint" type="fixed">
-  <origin xyz="0 0 0" rpy="0 0 0"/>
-  <parent link="chasis"/>
-  <child link="left_wheel"/>
-</joint>
 <!-- left side wheel -->
   <link name="left_wheel">
     <inertial>
+      <mass value="5"/>
       <origin xyz="0 0 0" rpy="0 1.5707 1.5707"/>
       <mass value="5.0"/>
@@ -119,6 +113,6 @@
   </joint>
  <joint type="continuous" name="right_wheel_hinge">
-    <origin xyz="0 0.15 0" rpy="0 0 0"/>
-    <child link="left_wheel"/>
+    <origin xyz="0 -0.15 0" rpy="0 0 0"/>
+    <child link="right_wheel"/>
     <parent link="chassis"/>
     <axis xyz="0 1 0" rpy="0 0 0"/>
@@ -126,8 +120,72 @@
     <dynamics damping="1.0" friction="1.0"/>
   </joint>
- <joint name="camera_joint" type="fixed">
-  <origin xyz="0 0 0" rpy="0 0 0"/>
-  <parent link="chasis"/>
-  <child link="left_wheel"/>
-</joint>
+  <link name="camera">
+    <collision>
+      <origin xyz="0 0 0" rpy="0 0 0"/>
+      <geometry>
+        <box size="0.05 0.05 0.05"/>
+      </geometry>
+    </collision>
+    <inertial>
+      <origin xyz="0 0 0" rpy="0 0 0"/>
+      <mass value="0.1"/>
+      <inertia
+            ixx="1e-6" ixy="0" ixz="0"
+            iyy="1e-6" iyz="0"
+            izz="1e-6"/>
+    </inertial>
+    <visual>
+      <origin xyz="0 0 0" rpy="0 0 0"/>
+      <geometry>
+        <box size="0.05 0.05 0.05"/>
+      </geometry>
+    </visual>
+  </link>
+  <joint name="camera_joint" type="fixed">
+    <origin xyz="0.2 0 0" rpy="0 0 0"/>
+    <parent link="chassis"/>
+    <child link="camera"/>
+    <axis xyz="0 1 0"/>
+  </joint>
+  <link name="hokuyo">
+        <collision>
+            <origin xyz="0 0 0" rpy="0 0 0"/>
+            <geometry>
+                <box size="0.1 0.1 0.1"/>
+            </geometry>
+        </collision>
+        <inertial>
+            <origin xyz="0 0 0" rpy="0 0 0"/>
+            <mass value="1e-5"/>
+            <inertia
+                ixx="1e-6" ixy="0" ixz="0"
+                iyy="1e-6" iyz="0"
+                izz="1e-6"
+                />
+        </inertial>
+        <visual>
+            <origin xyz="0 0 0" rpy="0 0 0"/>
+            <geometry>
+                <mesh filename="package://my_robot/meshes/hokuyo.dae"/>
+            </geometry>
+        </visual>
+    </link>
+    <joint name="hokuyo_joint" type="fixed">
+        <origin xyz="0.15 0 .1" rpy="0 0 0"/>
+        <axis xyz="0 1 0"/>
+        <parent link="chassis"/>
+        <child link="hokuyo"/>
+    </joint>
+    <gazebo reference="left_wheel">
+          <material>Gazebo/Green</material>
+    </gazebo>
+    <gazebo reference="right_wheel">
+        <material>Gazebo/Green</material>
+    </gazebo>
+     <gazebo reference="hokuyo">
+        <material>Gazebo/Red</material>
+    </gazebo>
+     <gazebo reference="chassis">
+        <material>Gazebo/Blue</material>
+    </gazebo>
 </robot>
